File: kle.pcb.kicad_pcb (KiCad board)
At the start: 2 copper layers, 191 parts, among them J2 Conn_02x03_Odd_Even, K0 Esc, K1 F1, K10 F10, K11 F11, K12 F12, K13 PrtSc,NmLk, K14 Pause,ScrLk, K15 Delete,Insert, K16 ~~,`, K17 !,1, K18 @,2, K19 #,3, K2 F2, K20 $,4, K21 %,5, K22 ^,6, K23 &,7, K24 *,8, K25 (,9, K26 ),0, K27 _,-, K28 +,=, K29 Backspace, K3 F3, K30 Home, K31 Tab, K32 Q, K33 W, K34 E, K35 R, K36 T, K37 Y, K38 U, K39 I, K4 F4, K40 O, K41 P, K42 {,[, K43 },], K44 |,\, K45 Page Up, K46 Caps Lock, K47 A, K48 S, K49 D, K5 F5, K50 F, K51 G, K52 H, K53 J, K54 K, K55 L, K56 :,;, K57 ",', K58 Enter, K59 Page Down, K6 F6, K60 Shift, K61 Z, K62 X, K63 C, K64 V, K65 B, K66 N, K67 M, K68 <,,, K69 >,., K7 F7, K70 ?,/, K71 Shift, K72 ↑, K73 End, K74 Ctrl, K75 Win, K76 Alt, K77 Blank, K78 Alt, K79 Fn, K8 F8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

Commit message: tweak layout
Parts:
- K77: value Blank -> Space
- moved H2 243.0 mm to (304.8, 123.8)
- moved C1 163.5 mm to (82.0, 183.7)
- moved C6 163.5 mm to (75.5, 186.7)
- moved C7 163.5 mm to (75.5, 199.7)
- moved C2 163.5 mm to (95.6, 187.4)
- moved C3 163.5 mm to (87.0, 201.5)
- moved C4 163.5 mm to (58.5, 188.0)
- moved C5 163.5 mm to (96.5, 198.5)
- moved C8 163.5 mm to (91.0, 201.5)
- moved D84 163.5 mm to (54.9, 187.0)
- moved D85 163.5 mm to (55.1, 185.5)
- moved P1 163.5 mm to (61.1, 182.6)
- moved R1 163.5 mm to (82.4, 201.5)
- moved R2 163.5 mm to (63.5, 187.9)
- moved R3 163.5 mm to (61.0, 187.9)
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Routing:
- net /Row_0: track 302.5 -> 0.00 mm
- net /Row_1: track 301.3 -> 0.00 mm
- net /Row_2: track 296.6 -> 0.00 mm
- net /Row_5: track 293.4 -> 0.00 mm
- net /Row_3: track 293.1 -> 0.00 mm
- net /Row_4: track 288.3 -> 0.00 mm
- net /Col_7: track 203.1 -> 0.00 mm, vias 5 -> 0
- net /Col_5: track 185.2 -> 0.00 mm, vias 6 -> 0
- net /Col_6: track 183.2 -> 0.00 mm, vias 5 -> 0
- net /Col_0: track 144.1 -> 0.00 mm
- net /Col_4: track 136.0 -> 0.00 mm, vias 5 -> 0
- net /Col_1: track 115.0 -> 0.00 mm, vias 5 -> 0
- net /Col_11: track 113.0 -> 0.00 mm, vias 6 -> 0
- net /Col_3: track 112.3 -> 0.00 mm, vias 5 -> 0
- net /Col_2: track 110.3 -> 0.00 mm, vias 6 -> 0
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
Commit message: progress
Parts:
- removed C6, C7: 22p, Capacitor_SMD:C_0805_2012Metric_Pad1.15x1.40mm_HandSolder
- removed C8: 1u, Capacitor_SMD:C_0805_2012Metric_Pad1.15x1.40mm_HandSolder
- removed D84, D85: PTVS5V0Z1USK, Diode_SMD:Nexperia_DSN1608-2_1.6x0.8mm
- removed J2: Conn_02x03_Odd_Even, Connector_PinHeader_2.54mm:PinHeader_2x03_P2.54mm_Vertical
- removed R1, R4: 10k, Resistor_SMD:R_0805_2012Metric_Pad1.15x1.40mm_HandSolder
- removed R2, R3: 22R, Resistor_SMD:R_0805_2012Metric_Pad1.15x1.40mm_HandSolder
- removed SW1: Reset_SW, Button_Switch_SMD:SW_Push_1P1T_NO_6x6mm_H9.5mm
- removed U1: ATmega32U4-AU, Package_QFP:TQFP-44_10x10mm_P0.8mm
- removed Y1: Crystal, Crystal:Crystal_SMD_5032-2Pin_5.0x3.2mm_HandSoldering
- added D86: SP0503BAHT, Package_TO_SOT_SMD:SOT-143, F.Cu at (44.8, 19.4)
- added R5: 22R, Resistor_SMD:R_0805_2012Metric_Pad1.20x1.40mm_HandSolder, F.Cu at (47.5, 19.6)
- added R6: 22R, Resistor_SMD:R_0805_2012Metric_Pad1.20x1.40mm_HandSolder, F.Cu at (42.0, 19.6)
- added U3: MDBT50Q-1MV2, RF_Module:Raytac_MDBT50Q, F.Cu at (42.8, 36.5)
- added Y2: Crystal, Crystal:Crystal_SMD_5032-2Pin_5.0x3.2mm_HandSoldering, B.Cu at (53.5, 35.8)
- C1, C2, C3, C4, C5: moved to F.Cu
- moved C3 184.5 mm to (57.2, 19.4), turned to 90 degrees
- moved C5 182.1 mm to (63.1, 19.4)
- moved C2 173.0 mm to (54.2, 19.4), turned to 90 degrees
- moved C4 168.6 mm to (60.1, 19.4), turned to 90 degrees
- moved P1 167.6 mm to (44.6, 15.8)
- moved C1 167.1 mm to (51.3, 19.4), turned to 90 degrees
Routing:
- net /Row_0: track 0.00 -> 463.8 mm, vias 0 -> 5
- net /Row_1: track 0.00 -> 364.9 mm, vias 0 -> 14
- net /Row_2: track 0.00 -> 360.9 mm, vias 0 -> 13
- net /Row_3: track 0.00 -> 325.5 mm, vias 0 -> 13
- net /Row_4: track 0.00 -> 316.2 mm, vias 0 -> 10
- net /Row_5: track 0.00 -> 299.3 mm, vias 0 -> 3
- net /Col_2: track 0.00 -> 123.0 mm
- net /Col_13: track 0.00 -> 116.9 mm
- net /Col_14: track 0.00 -> 116.3 mm
- net /Col_1: track 0.00 -> 113.7 mm
- net /Col_11: track 0.00 -> 113.7 mm
- net /Col_10: track 0.00 -> 111.5 mm
- net /Col_9: track 0.00 -> 107.8 mm
- net /Col_5: track 0.00 -> 106.1 mm
- net /Col_0: track 0.00 -> 104.2 mm
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
Commit message: progress
Parts:
- added C10: 22p, Capacitor_SMD:C_0805_2012Metric_Pad1.18x1.45mm_HandSolder, F.Cu at (130.0, 120.2)
- added C9: 22p, Capacitor_SMD:C_0805_2012Metric_Pad1.18x1.45mm_HandSolder, F.Cu at (130.0, 118.2)
- Y2: footprint Crystal:Crystal_SMD_5032-2Pin_5.0x3.2mm_HandSoldering -> Crystal:Crystal_SMD_2012-2Pin_2.0x1.2mm_HandSoldering; moved to F.Cu
- moved U3 131.6 mm to (142.8, 122.0), turned to -90 degrees
- moved Y2 115.2 mm to (133.1, 119.2), turned to -90 degrees
- moved H2 40.1 mm to (324.0, 159.0)
Connections:
- D86 pad 3: Net-(P1-D-) -> Net-(P1-D+)
- D86 pad 4: Net-(P1-D+) -> Net-(P1-D-)
Routing:
- net /Row_0: track 463.8 -> 0.14 mm, vias 5 -> 0
- net /Row_1: track 364.9 -> 0.00 mm, vias 14 -> 0
- net /Row_2: track 360.9 -> 0.00 mm, vias 13 -> 0
- net /Row_3: track 325.5 -> 0.00 mm, vias 13 -> 0
- net /Row_4: track 316.2 -> 0.00 mm, vias 10 -> 0
- net /Row_5: track 299.3 -> 471.3 mm, vias 3 -> 0
- net /D-: track 17.1 -> 156.4 mm
- net /D+: track 24.3 -> 156.3 mm, vias 2 -> 0
- net /Col_0: track 104.2 -> 123.2 mm
- net /Col_7: track 99.2 -> 86.1 mm
- net /Col_2: track 123.0 -> 110.0 mm
- net VCC: track 35.2 -> 22.6 mm, vias 0 -> 1
- net /Col_14: track 116.3 -> 105.1 mm
- net /Col_8: track 96.3 -> 86.1 mm
- net Net-(D59-A): track 0.00 -> 10.2 mm
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