File: kle.pcb.kicad_pcb (KiCad board)
At the start: 2 copper layers, 185 parts, among them K0 Esc, K1 F1, K10 F10, K11 F11, K12 F12, K13 PrtSc,NmLk, K14 Pause,ScrLk, K15 Delete,Insert, K16 ~~,`, K17 !,1, K18 @,2, K19 #,3, K2 F2, K20 $,4, K21 %,5, K22 ^,6, K23 &,7, K24 *,8, K25 (,9, K26 ),0, K27 _,-, K28 +,=, K29 Backspace, K3 F3, K30 Home, K31 Tab, K32 Q, K33 W, K34 E, K35 R, K36 T, K37 Y, K38 U, K39 I, K4 F4, K40 O, K41 P, K42 {,[, K43 },], K44 |,\, K45 Page Up, K46 Caps Lock, K47 A, K48 S, K49 D, K5 F5, K50 F, K51 G, K52 H, K53 J, K54 K, K55 L, K56 :,;, K57 ",', K58 Enter, K59 Page Down, K6 F6, K60 Shift, K61 Z, K62 X, K63 C, K64 V, K65 B, K66 N, K67 M, K68 <,,, K69 >,., K7 F7, K70 ?,/, K71 Shift, K72 ↑, K73 End, K74 Ctrl, K75 Win, K76 Alt, K77 Space, K78 Alt, K79 Fn, K8 F8, K80 Ctrl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

Commit message: progress
Parts:
- K75: value Win -> Lin
- moved H4 285.7 mm to (295.6, 47.5)
- moved H3 202.7 mm to (78.6, 38.9)
- moved H1 124.9 mm to (76.2, 104.7)
- moved R5 110.2 mm to (157.7, 19.2)
- moved P1 110.0 mm to (154.7, 15.3)
- moved D86 109.9 mm to (154.7, 19.0)
- moved C5 109.8 mm to (172.9, 19.1)
- moved C1 109.8 mm to (161.1, 19.1)
- moved C3 109.8 mm to (167.0, 19.1)
- moved C2 109.8 mm to (164.0, 19.1)
- moved C4 109.8 mm to (169.9, 19.1)
- moved R6 109.7 mm to (151.7, 19.2)
- moved H2 58.3 mm to (304.4, 104.1)
- moved C9 26.5 mm to (155.4, 125.7), turned to 0 degrees
- moved C10 25.6 mm to (155.4, 123.7), turned to 0 degrees
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Connections:
- D86 pad 3: Net-(P1-D+) -> Net-(P1-D-)
- D86 pad 4: Net-(P1-D-) -> Net-(P1-D+)
- U3 pad 10: unconnected-(U3-P0.29-Pad10) -> /Col_11
- U3 pad 14: unconnected-(U3-P0.30-Pad14) -> /Col_10
- U3 pad 16: unconnected-(U3-P0.27-Pad16) -> /Col_9
- U3 pad 19: unconnected-(U3-P0.26-Pad19) -> /Col_7
- U3 pad 20: unconnected-(U3-P0.04-Pad20) -> /Col_5
- U3 pad 22: unconnected-(U3-P0.06-Pad22) -> /Row_3
- U3 pad 24: unconnected-(U3-P0.08-Pad24) -> /Row_0
- U3 pad 26: unconnected-(U3-P1.09-Pad26) -> /Row_1
- U3 pad 27: unconnected-(U3-P0.11-Pad27) -> /Row_2
- U3 pad 29: unconnected-(U3-P0.12-Pad29) -> /Col_6
- U3 pad 3: unconnected-(U3-P1.10-Pad3) -> /Row_5
- U3 pad 37: unconnected-(U3-P0.13-Pad37) -> /Col_12
- U3 pad 4: unconnected-(U3-P1.11-Pad4) -> /Col_15
- U3 pad 46: unconnected-(U3-P0.22-Pad46) -> /Col_4
- U3 pad 48: unconnected-(U3-P0.24-Pad48) -> /Row_4
- U3 pad 49: unconnected-(U3-P0.25-Pad49) -> /Col_3
- U3 pad 50: unconnected-(U3-P1.02-Pad50) -> /Col_2
- U3 pad 52: unconnected-(U3-P0.09-Pad52) -> /Col_0
- U3 pad 54: unconnected-(U3-P0.10-Pad54) -> /Col_1
- U3 pad 6: unconnected-(U3-P1.13-Pad6) -> /Col_14
- U3 pad 7: unconnected-(U3-P1.14-Pad7) -> /Col_8
- U3 pad 8: unconnected-(U3-P1.15-Pad8) -> /Col_13
Routing:
- net /Row_0: track 0.14 -> 542.4 mm, vias 0 -> 3
- net /Row_1: track 0.00 -> 521.8 mm, vias 0 -> 3
- net /Row_2: track 0.00 -> 500.3 mm, vias 0 -> 3
- net /Row_3: track 0.00 -> 479.7 mm, vias 0 -> 3
- net /Row_4: track 0.00 -> 281.4 mm, vias 0 -> 1
- net /Col_15: track 95.2 -> 289.2 mm, vias 0 -> 7
- net /Row_5: track 471.3 -> 286.3 mm, vias 0 -> 1
- net /Col_12: track 42.0 -> 225.8 mm, vias 0 -> 5
- net /Col_14: track 105.1 -> 277.5 mm, vias 0 -> 3
- net /Col_13: track 109.4 -> 257.1 mm, vias 0 -> 5
- net /Col_11: track 113.0 -> 243.0 mm, vias 0 -> 6
- net VCC: track 22.6 -> 143.1 mm, vias 1 -> 3
- net /Col_10: track 107.1 -> 215.8 mm, vias 0 -> 8
- net /Col_9: track 107.1 -> 195.8 mm, vias 0 -> 8
- net /Col_8: track 86.1 -> 172.3 mm, vias 0 -> 7
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
Commit message: progress
Parts:
- added D84: LED, LED_SMD:LED_0805_2012Metric_Pad1.15x1.40mm_HandSolder, F.Cu at (196.4, 118.3)
- added JP1: Jumper_2_Open, Jumper:SolderJumper-2_P1.3mm_Open_TrianglePad1.0x1.5mm, F.Cu at (186.3, 123.8)
- added R1: 10k, Resistor_SMD:R_0805_2012Metric_Pad1.20x1.40mm_HandSolder, F.Cu at (192.5, 118.3)
- added R2: 22R, Resistor_SMD:R_0805_2012Metric_Pad1.20x1.40mm_HandSolder, F.Cu at (184.2, 119.2)
- added R3: 22R, Resistor_SMD:R_0805_2012Metric_Pad1.20x1.40mm_HandSolder, F.Cu at (184.2, 117.1)
- added R4: 22R, Resistor_SMD:R_0805_2012Metric_Pad1.20x1.40mm_HandSolder, F.Cu at (189.1, 123.1)
- added R7: 22R, Resistor_SMD:R_0805_2012Metric_Pad1.20x1.40mm_HandSolder, F.Cu at (145.6, 132.1)
- added U2: BQ24075RGT, Package_DFN_QFN:VQFN-16-1EP_3x3mm_P0.5mm_EP1.6x1.6mm, F.Cu at (188.4, 118.5)
Routing:
- net VCC: track 143.1 -> 181.8 mm, vias 3 -> 5
- net /Reset: track 0.00 -> 17.3 mm
- net Net-(JP1-A): track 0.00 -> 10.2 mm
- net Net-(D84-K): track 0.00 -> 8.05 mm
- net Net-(U2-TS): track 0.00 -> 2.44 mm
- net Net-(JP1-B): track 0.00 -> 2.19 mm
- net Net-(D84-A): track 0.00 -> 1.88 mm
- net VDDH: track 0.00 -> 1.68 mm

Commit message: add battery connector
Parts:
- added J1: Conn_01x02_Socket, Connector_JST:JST_EH_S2B-EH_1x02_P2.50mm_Horizontal, B.Cu at (201.8, 121.7)
Routing:
- net +BATT: track 0.00 -> 19.0 mm, vias 0 -> 2
- net VDDH: track 1.68 -> 9.24 mm, vias 0 -> 2
- net Net-(D84-K): track 8.05 -> 8.76 mm

Commit message: save footprint positions
Parts:
- added SW1: SW_SPST, Button_Switch_SMD:SW_SPST_TS-1088-xR025, F.Cu at (130.5, 122.4)
- H1, H2, H3, H4: footprint MountingHole:MountingHole_3.2mm_M3_DIN965 -> MountingHole:MountingHole_3.2mm_M3_DIN965_Pad
- P1: footprint Connector_USB:USB_C_Plug_Molex_105444 -> footprints:CONN_8p94X6p5X3p16_12L_GCC; moved to B.Cu
- moved R7 19.7 mm to (130.4, 119.6), turned to 180 degrees
- moved P1 2.23 mm to (154.7, 13.1)
Connections:
- J1 pad 2: GND -> -BATT
Routing:
- net VCC: track 182.2 -> 201.8 mm, vias 5 -> 7
- net /Reset: track 17.3 -> 24.2 mm, vias 0 -> 2
- net GND: track 13.8 -> 9.09 mm, vias 3 -> 2
- net Net-(P1-D-): track 4.69 -> 3.54 mm, vias 0 -> 1
- net Net-(P1-D+): track 4.69 -> 3.54 mm, vias 0 -> 1
- net /Col_2: track 154.1 -> 154.6 mm
- net /Col_6: vias 8 -> 7
