File: kle.pcb.kicad_pcb (KiCad board)
At the start: 2 copper layers, 195 parts, among them J1 Conn_01x02_Socket, K0 Esc, K1 F1, K10 F10, K11 F11, K12 F12, K13 PrtSc,NmLk, K14 Pause,ScrLk, K15 Delete,Insert, K16 ~~,`, K17 !,1, K18 @,2, K19 #,3, K2 F2, K20 $,4, K21 %,5, K22 ^,6, K23 &,7, K24 *,8, K25 (,9, K26 ),0, K27 _,-, K28 +,=, K29 Backspace, K3 F3, K30 Home, K31 Tab, K32 Q, K33 W, K34 E, K35 R, K36 T, K37 Y, K38 U, K39 I, K4 F4, K40 O, K41 P, K42 {,[, K43 },], K44 |,\, K45 Page Up, K46 Caps Lock, K47 A, K48 S, K49 D, K5 F5, K50 F, K51 G, K52 H, K53 J, K54 K, K55 L, K56 :,;, K57 ",', K58 Enter, K59 Page Down, K6 F6, K60 Shift, K61 Z, K62 X, K63 C, K64 V, K65 B, K66 N, K67 M, K68 <,,, K69 >,., K7 F7, K70 ?,/, K71 Shift, K72 ↑, K73 End, K74 Ctrl, K75 Lin, K76 Alt, K77 Space, K78 Alt, K79 Fn, K8 F8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

Commit message: fix board generation
Routing:
- net /Reset: track 24.2 -> 35.7 mm

Commit message: add usb bump
Routing:
- removed copper zone on B.Cu, net GND
- removed copper zone on F.Cu, net GND
Changed lines of the file:
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@@
 		(net 153)
-	)
-	(zone
-		(net 1)
-		(net_name "GND")
-		(layers "F.Cu" "B.Cu")
-		(hatch edge 0.5)
-		(connect_pads
-			(clearance 0)
-		)
-		(min_thickness 0.25)
-		(filled_areas_thickness no)
-		(fill yes
-			(thermal_gap 0)
-			(thermal_bridge_width 0)
-		)
-		(polygon
-			(pts
-				(xy 39 10.575) (xy 346.75 10.575) (xy 346.75 133.824999) (xy 39 133.824999)
-			)
-		)
-	)
-	(zone
-		(net 1)
-		(net_name "GND")
-		(layers "F.Cu" "B.Cu")
-		(hatch edge 0.5)
-		(connect_pads
-			(clearance 0)
-		)
-		(min_thickness 0.25)
-		(filled_areas_thickness no)
-		(fill yes
-			(thermal_gap 0)
-			(thermal_bridge_width 0)
-		)
-		(polygon
-			(pts
-				(xy 39 10.575) (xy 346.75 10.575) (xy 346.75 133.824999) (xy 39 133.824999)
-			)
-		)
-	)
-	(zone
-		(net 0)
-		(net_name "")
-		(layer "Edge.Cuts")
-		(hatch edge 0.5)
-		(connect_pads
-			(clearance 0)
-		)
-		(min_thickness 0.25)
-		(filled_areas_thickness no)
-		(fill yes
-			(thermal_gap 0)
-			(thermal_bridge_width 0)
-		)
-		(polygon
-			(pts
-				(xy 39 10.575) (xy 346.75 10.575) (xy 346.75 133.824999) (xy 39 133.824999)
-			)
-		)
-	)
-	(zone
-		(net 0)
-		(net_name "")
-		(layer "Edge.Cuts")
-		(hatch edge 0.5)
-		(connect_pads
-			(clearance 0)
-		)
-		(min_thickness 0.25)
-		(filled_areas_thickness no)
-		(fill yes
-			(thermal_gap 0)
-			(thermal_bridge_width 0)
-		)
-		(polygon
-			(pts
-				(xy 39 10.575) (xy 346.75 10.575) (xy 346.75 133.824999) (xy 39 133.824999)
-			)
-		)
 	)
 	(embedded_fonts no)
