File: kle.pcb.kicad_sch (KiCad schematic)
At the start: 191 parts, among them J2 Conn_02x03_Odd_Even, K0 Esc, K1 F1, K10 F10, K11 F11, K12 F12, K13 PrtSc,NmLk, K14 Pause,ScrLk, K15 Delete,Insert, K16 ~~,`, K17 !,1, K18 @,2, K19 #,3, K2 F2, K20 $,4, K21 %,5, K22 ^,6, K23 &,7, K24 *,8, K25 (,9, K26 ),0, K27 _,-, K28 +,=, K29 Backspace, K3 F3, K30 Home, K31 Tab, K32 Q, K33 W, K34 E, K35 R, K36 T, K37 Y, K38 U, K39 I, K4 F4, K40 O, K41 P, K42 {,[, K43 },], K44 |,\, K45 Page Up, K46 Caps Lock, K47 A, K48 S, K49 D, K5 F5, K50 F, K51 G, K52 H, K53 J, K54 K, K55 L, K56 :,;, K57 ",', K58 Enter, K59 Page Down, K6 F6, K60 Shift, K61 Z, K62 X, K63 C, K64 V, K65 B, K66 N, K67 M, K68 <,,, K69 >,., K7 F7, K70 ?,/, K71 Shift, K72 ↑, K73 End, K74 Ctrl, K75 Win, K76 Alt, K77 Blank, K78 Alt, K79 Fn, K8 F8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

Commit message: initial commit
Parts:
- K77: value Blank -> Space
Changed lines of the file:
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@@
 			)
 		)
-		(property "Value" "Blank"
+		(property "Value" "Space"
 			(at 160.02 92.71 0)
 			(effects

Commit message: progress
Parts:
- removed C6, C7: 22p, Capacitor_SMD:C_0805_2012Metric_Pad1.15x1.40mm_HandSolder, symbol Device:C
- removed C8: 1u, Capacitor_SMD:C_0805_2012Metric_Pad1.15x1.40mm_HandSolder, symbol Device:C
- removed D84, D85: PTVS5V0Z1USK, Diode_SMD:Nexperia_DSN1608-2_1.6x0.8mm, symbol Diode:PTVS5V0Z1USK
- removed J2: Conn_02x03_Odd_Even, Connector_PinHeader_2.54mm:PinHeader_2x03_P2.54mm_Vertical, symbol Connector_Generic:Conn_02x03_Odd_Even
- removed R1, R4: 10k, Resistor_SMD:R_0805_2012Metric_Pad1.15x1.40mm_HandSolder, symbol Device:R
- removed R2, R3: 22R, Resistor_SMD:R_0805_2012Metric_Pad1.15x1.40mm_HandSolder, symbol Device:R
- removed SW1: Reset_SW, Button_Switch_SMD:SW_Push_1P1T_NO_6x6mm_H9.5mm, symbol Switch:SW_Push
- removed U1: ATmega32U4-AU, Package_QFP:TQFP-44_10x10mm_P0.8mm, symbol MCU_Microchip_ATmega:ATmega32U4-A
- removed Y1: Crystal, Crystal:Crystal_SMD_5032-2Pin_5.0x3.2mm_HandSoldering, symbol Device:Crystal
- added C10, C9: 22p, Capacitor_SMD:C_0805_2012Metric_Pad1.15x1.40mm_HandSolder, symbol Device:C
- added D86: SP0503BAHT, Package_TO_SOT_SMD:SOT-143, symbol Power_Protection:SP0503BAHT
- added R5, R6: 22R, Resistor_SMD:R_0805_2012Metric_Pad1.20x1.40mm_HandSolder, symbol Device:R
- added U3: MDBT50Q-1MV2, RF_Module:Raytac_MDBT50Q, symbol RF_Module:MDBT50Q-1MV2
- added Y2: Crystal, Crystal:Crystal_SMD_5032-2Pin_5.0x3.2mm_HandSoldering, symbol Device:Crystal
Connections:
- net GND: now also C10.2, C9.2, D86.1 (A), U3.1 (GND), U3.15 (GND), U3.2 (GND), U3.33 (GND), U3.55 (GND)
- net Reset: now also U3.40 (P0.18)
- net VCC: now also D86.2 (K), U3.30 (VDDH), U3.32 (VBUS)
- net at P1.A7 (D-): now also D86.3 (K), R5.2
- net at P1.A6 (D+): now also D86.4 (K), R6.2
- new net D+: R6.1, U3.35 (D+)
- new net D-: R5.1, U3.34 (D-)
- new net X1: C9.1, U3.17 (P0.00), Y2.1
- new net X2: C10.1, U3.18 (P0.01), Y2.2
- no-connect marks 0 -> 1
Other:
- moved on the sheet: P1

Commit message: progress
Parts:
- C10, C9: footprint Capacitor_SMD:C_0805_2012Metric_Pad1.15x1.40mm_HandSolder -> Capacitor_SMD:C_0805_2012Metric_Pad1.18x1.45mm_HandSolder
- Y2: footprint Crystal:Crystal_SMD_5032-2Pin_5.0x3.2mm_HandSoldering -> Crystal:Crystal_SMD_2012-2Pin_2.0x1.2mm_HandSoldering
Connections:
- net at P1.A7 (D-), R5.2: now also D86.4 (K); no longer D86.3 (K)
- net at P1.A6 (D+), R6.2: now also D86.3 (K); no longer D86.4 (K)
Changed lines of the file:
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@@
 	)
 	(junction
-		(at 175.26 241.3)
+		(at 170.18 241.3)
 		(diameter 0)
 		(color 0 0 0 0)
@@
 	)
 	(junction
+		(at 175.26 243.84)
+		(diameter 0)
+		(color 0 0 0 0)
+	)
+	(junction
 		(at 101.6 271.78)
 		(diameter 0)
@@
 		(color 0 0 0 0)
 	)
-	(junction
-		(at 170.18 243.84)
-		(diameter 0)
-		(color 0 0 0 0)
-	)
 	(no_connect
 		(at 246.38 163.83)
@@
 	(wire
 		(pts
-			(xy 175.26 241.3) (xy 175.26 250.19)
+			(xy 246.38 168.91) (xy 243.84 168.91)
 		)
 		(stroke
@@
 	(wire
 		(pts
-			(xy 246.38 168.91) (xy 243.84 168.91)
+			(xy 25.4 252.73) (xy 25.4 261.62)
 		)
 		(stroke
@@
 	(wire
 		(pts
-			(xy 25.4 252.73) (xy 25.4 261.62)
+			(xy 170.18 237.49) (xy 170.18 241.3)
 		)
 		(stroke
@@
 	(wire
 		(pts
+			(xy 193.04 241.3) (xy 170.18 241.3)
+		)
+		(stroke
+			(width 0)
+			(type default)
+		)
+	)
+	(wire
+		(pts
 			(xy 243.84 166.37) (xy 243.84 168.91)
 		)
@@
 	(wire
 		(pts
-			(xy 195.58 265.43) (xy 195.58 273.05)
+			(xy 175.26 243.84) (xy 175.26 250.19)
 		)
 		(stroke
@@
 	(wire
 		(pts
-			(xy 93.98 256.54) (xy 97.79 256.54)
+			(xy 195.58 265.43) (xy 195.58 273.05)
 		)
 		(stroke
@@
 	(wire
 		(pts
-			(xy 157.48 250.19) (xy 157.48 246.38)
+			(xy 93.98 256.54) (xy 97.79 256.54)
 		)
 		(stroke
@@
 	(wire
 		(pts
-			(xy 175.26 241.3) (xy 193.04 241.3)
+			(xy 157.48 250.19) (xy 157.48 246.38)
 		)
 		(stroke
@@
 	(wire
 		(pts
-			(xy 170.18 243.84) (xy 193.04 243.84)
+			(xy 170.18 241.3) (xy 170.18 250.19)
 		)
 		(stroke
@@
 	(wire
 		(pts
-			(xy 93.98 251.46) (xy 93.98 256.54)
+			(xy 175.26 237.49) (xy 175.26 243.84)
 		)
 		(stroke
@@
 	(wire
 		(pts
-			(xy 165.1 246.38) (xy 193.04 246.38)
+			(xy 93.98 251.46) (xy 93.98 256.54)
 		)
 		(stroke
@@
 	(wire
 		(pts
-			(xy 294.64 189.23) (xy 294.64 191.77)
+			(xy 165.1 246.38) (xy 193.04 246.38)
 		)
 		(stroke
@@
 	(wire
 		(pts
-			(xy 59.69 261.62) (xy 71.12 261.62)
+			(xy 294.64 189.23) (xy 294.64 191.77)
 		)
 		(stroke
@@
 	(wire
 		(pts
-			(xy 48.26 261.62) (xy 59.69 261.62)
+			(xy 59.69 261.62) (xy 71.12 261.62)
 		)
 		(stroke
@@
 	(wire
 		(pts
-			(xy 287.02 146.05) (xy 287.02 148.59)
+			(xy 48.26 261.62) (xy 59.69 261.62)
 		)
 		(stroke
@@
 	(wire
 		(pts
-			(xy 105.41 256.54) (xy 109.22 256.54)
+			(xy 287.02 146.05) (xy 287.02 148.59)
 		)
 		(stroke
@@
 	(wire
 		(pts
-			(xy 170.18 243.84) (xy 170.18 250.19)
+			(xy 105.41 256.54) (xy 109.22 256.54)
 		)
 		(stroke
@@
 	(wire
 		(pts
-			(xy 175.26 237.49) (xy 175.26 241.3)
-		)
-		(stroke
-			(width 0)
-			(type default)
-		)
-	)
-	(wire
-		(pts
 			(xy 59.69 269.24) (xy 71.12 269.24)
 		)
@@
 	(wire
 		(pts
-			(xy 170.18 237.49) (xy 170.18 243.84)
+			(xy 259.08 144.78) (xy 259.08 148.59)
 		)
 		(stroke
@@
 	(wire
 		(pts
-			(xy 259.08 144.78) (xy 259.08 148.59)
+			(xy 175.26 243.84) (xy 193.04 243.84)
 		)
 		(stroke
@@
 			)
 		)
-		(property "Footprint" "Capacitor_SMD:C_0805_2012Metric_Pad1.15x1.40mm_HandSolder"
+		(property "Footprint" "Capacitor_SMD:C_0805_2012Metric_Pad1.18x1.45mm_HandSolder"
 			(at 94.9452 269.24 0)
 			(effects
@@
 			)
 		)
-		(property "Footprint" "Capacitor_SMD:C_0805_2012Metric_Pad1.15x1.40mm_HandSolder"
+		(property "Footprint" "Capacitor_SMD:C_0805_2012Metric_Pad1.18x1.45mm_HandSolder"
 			(at 110.1852 269.24 0)
 			(effects
@@
 			)
 		)
-		(property "Footprint" "Crystal:Crystal_SMD_5032-2Pin_5.0x3.2mm_HandSoldering"
+		(property "Footprint" "Crystal:Crystal_SMD_2012-2Pin_2.0x1.2mm_HandSoldering"
 			(at 101.6 256.54 0)
 			(effects

Commit message: progress
Parts:
- K75: value Win -> Lin
Connections:
- net Col_0: now also U3.52 (P0.09)
- net Col_1: now also U3.54 (P0.10)
- net Col_10: now also U3.14 (P0.30)
- net Col_11: now also U3.10 (P0.29)
- net Col_12: now also U3.37 (P0.13)
- net Col_13: now also U3.8 (P1.15)
- net Col_14: now also U3.6 (P1.13)
- net Col_15: now also U3.4 (P1.11)
- net Col_2: now also U3.50 (P1.02)
- net Col_3: now also U3.49 (P0.25)
- net Col_4: now also U3.46 (P0.22)
- net Col_5: now also U3.20 (P0.04)
- net Col_6: now also U3.29 (P0.12)
- net Col_7: now also U3.19 (P0.26)
- net Col_8: now also U3.7 (P1.14)
- net Col_9: now also U3.16 (P0.27)
- net Row_0: now also U3.24 (P0.08)
- net Row_1: now also U3.26 (P1.09)
- net Row_2: now also U3.27 (P0.11)
- net Row_3: now also U3.22 (P0.06)
- net Row_4: now also U3.48 (P0.24)
- net Row_5: now also U3.3 (P1.10)
- net at P1.A7 (D-), R5.2: now also D86.3 (K); no longer D86.4 (K)
- net at P1.A6 (D+), R6.2: now also D86.4 (K); no longer D86.3 (K)
- no-connect marks 1 -> 4

Commit message: progress
Parts:
- added C6, C7: 0.1u, Capacitor_SMD:C_0805_2012Metric_Pad1.15x1.40mm_HandSolder, symbol Device:C
- added C8: 22p, Capacitor_SMD:C_0805_2012Metric_Pad1.15x1.40mm_HandSolder, symbol Device:C
- added D84: LED, LED_SMD:LED_0805_2012Metric_Pad1.15x1.40mm_HandSolder, symbol Device:LED
- added JP1: Jumper_2_Open, Jumper:SolderJumper-2_P1.3mm_Open_TrianglePad1.0x1.5mm, symbol Jumper:Jumper_2_Open
- added R1: 10k, Resistor_SMD:R_0805_2012Metric_Pad1.20x1.40mm_HandSolder, symbol Device:R
- added R2, R3, R4, R7: 22R, Resistor_SMD:R_0805_2012Metric_Pad1.20x1.40mm_HandSolder, symbol Device:R
- added SW1: SW_SPST, symbol Switch:SW_SPST
- added U2: BQ24075RGT, Package_DFN_QFN:VQFN-16-1EP_3x3mm_P0.5mm_EP1.6x1.6mm, symbol Battery_Management:BQ24075RGT
- C10, C9: footprint Capacitor_SMD:C_0805_2012Metric_Pad1.18x1.45mm_HandSolder -> Capacitor_SMD:C_0805_2012Metric_Pad1.15x1.40mm_HandSolder
Connections:
- net GND: now also C6.2, C7.2, R2.2, R3.2, R4.2, R7.2, U2.15 (SYSOFF), U2.17 (VSS), U2.4 (~{CE}), U2.5 (EN2), U2.8 (VSS)
- net Reset: now also C8.2, R7.1, SW1.1 (A)
- net VCC: now also C6.1, C8.1, SW1.2 (B), U2.13 (IN)
- new net: JP1.2 (B), R4.1
- new net: R2.1, U2.1 (TS)
- new net: D84.1 (K), U2.9 (~{CHG})
- new net: D84.2 (A), R1.1
- new net: JP1.1 (A), R3.1, U2.16 (ISET)
- new net +BATT: U2.2 (BAT), U2.3 (BAT)
- new net VDDH: C7.1, R1.2, U2.10 (OUT), U2.11 (OUT), U2.6 (EN1)
- no-connect marks 4 -> 7

Commit message: add battery connector
Parts:
- added J1: Conn_01x02_Socket, Connector_JST:JST_EH_S2B-EH_1x02_P2.50mm_Horizontal, symbol Connector:Conn_01x02_Socket
Connections:
- net +BATT: now also J1.1 (Pin_1)
- new net -BATT: J1.2 (Pin_2)
Changed lines of the file:
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@@
 	)
 	(symbol
+		(lib_id "power:+BATT")
+		(at 102.87 222.25 90)
+		(unit 1)
+		(exclude_from_sim no)
+		(in_bom yes)
+		(on_board yes)
+		(dnp no)
+		(property "Reference" "#PWR021"
+			(at 106.68 222.25 0)
+			(effects
+				(font
+					(size 1.27 1.27)
+				)
+				(hide yes)
+			)
+		)
+		(property "Value" "+BATT"
+			(at 102.616 220.472 90)
+			(effects
+				(font
+					(size 1.27 1.27)
+				)
+				(justify left)
+			)
+		)
+		(property "Footprint" ""
+			(at 102.87 222.25 0)
+			(effects
+				(font
+					(size 1.27 1.27)
+				)
+				(hide yes)
+			)
+		)
+		(property "Datasheet" ""
+			(at 102.87 222.25 0)
+			(effects
+				(font
+					(size 1.27 1.27)
+				)
+				(hide yes)
+			)
+		)
+		(property "Description" "Power symbol creates a global label with name \"+BATT\""
+			(at 102.87 222.25 0)
+			(effects
+				(font
+					(size 1.27 1.27)
+				)
+				(hide yes)
+			)
+		)
+		(pin "1"
+		)
+		(instances
+			(project "kle.pcb"
+				(path "/a7762a06-9113-4833-9fbd-2a782c9e6227"
+					(reference "#PWR021")
+					(unit 1)
+				)
+			)
+		)
+	)
+	(symbol
 		(lib_id "Device:D")
 		(at 340.36 68.58 90)
@@
 	)
 	(symbol
+		(lib_id "Connector:Conn_01x02_Socket")
+		(at 107.95 222.25 0)
+		(unit 1)
+		(exclude_from_sim no)
+		(in_bom yes)
+		(on_board yes)
+		(dnp no)
+		(fields_autoplaced yes)
+		(property "Reference" "J1"
+			(at 109.22 222.2499 0)
+			(effects
+				(font
+					(size 1.27 1.27)
+				)
+				(justify left)
+			)
+		)
+		(property "Value" "Conn_01x02_Socket"
+			(at 109.22 224.7899 0)
+			(effects
+				(font
+					(size 1.27 1.27)
+				)
+				(justify left)
+			)
+		)
+		(property "Footprint" "Connector_JST:JST_EH_S2B-EH_1x02_P2.50mm_Horizontal"
+			(at 107.95 222.25 0)
+			(effects
+				(font
+					(size 1.27 1.27)
+				)
+				(hide yes)
+			)
+		)
+		(property "Datasheet" "~"
+			(at 107.95 222.25 0)
+			(effects
+				(font
+					(size 1.27 1.27)
+				)
+				(hide yes)
+			)
+		)
+		(property "Description" "Generic connector, single row, 01x02, script generated"
+			(at 107.95 222.25 0)
+			(effects
+				(font
+					(size 1.27 1.27)
+				)
+				(hide yes)
+			)
+		)
+		(pin "2"
+		)
+		(pin "1"
+		)
+		(instances
+			(project ""
+				(path "/a7762a06-9113-4833-9fbd-2a782c9e6227"
+					(reference "J1")
+					(unit 1)
+				)
+			)
+		)
+	)
+	(symbol
 		(lib_id "Device:D")
 		(at 314.96 55.88 90)
@@
 					(unit 1)
 				)
+			)
+		)
+	)
+	(symbol
+		(lib_id "power:+BATT")
+		(at 102.87 224.79 90)
+		(unit 1)
+		(exclude_from_sim no)
+		(in_bom yes)
+		(on_board yes)
+		(dnp no)
+		(property "Reference" "#PWR022"
+			(at 106.68 224.79 0)
+			(effects
+				(font
+					(size 1.27 1.27)
+				)
+				(hide yes)
+			)
+		)
+		(property "Value" "-BATT"
+			(at 102.87 226.822 90)
+			(effects
+				(font
+					(size 1.27 1.27)
+				)
+				(justify left)
+			)
+		)
+		(property "Footprint" ""
+			(at 102.87 224.79 0)
+			(effects
+				(font
+					(size 1.27 1.27)
+				)
+				(hide yes)
+			)
+		)
+		(property "Datasheet" ""
+			(at 102.87 224.79 0)
+			(effects
+				(font
+					(size 1.27 1.27)
+				)
+				(hide yes)
+			)
+		)
+		(property "Description" "Power symbol creates a global label with name \"+BATT\""
+			(at 102.87 224.79 0)
+			(effects
+				(font
+					(size 1.27 1.27)
+				)
+				(hide yes)
+			)
+		)
+		(pin "1"
+		)
+		(instances
+			(project "kle.pcb"
+				(path "/a7762a06-9113-4833-9fbd-2a782c9e6227"
+					(reference "#PWR022")
+					(unit 1)
+				)

Commit message: save footprint positions
Parts:
- H1, H2, H3, H4: footprint MountingHole:MountingHole_3.2mm_M3_DIN965 -> MountingHole:MountingHole_3.2mm_M3_DIN965_Pad
- P1: footprint Connector_USB:USB_C_Plug_Molex_105444 -> footprints:CONN_8p94X6p5X3p16_12L_GCC
- SW1: footprint (none) -> Button_Switch_SMD:SW_SPST_TS-1088-xR025
Changed lines of the file:
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@@
 			)
 		)
-		(property "Footprint" "MountingHole:MountingHole_3.2mm_M3_DIN965"
+		(property "Footprint" "MountingHole:MountingHole_3.2mm_M3_DIN965_Pad"
 			(at 30.48 232.41 0)
 			(effects
@@
 			)
 		)
-		(property "Footprint" "MountingHole:MountingHole_3.2mm_M3_DIN965"
+		(property "Footprint" "MountingHole:MountingHole_3.2mm_M3_DIN965_Pad"
 			(at 30.48 220.98 0)
 			(effects
@@
 			)
 		)
-		(property "Footprint" "MountingHole:MountingHole_3.2mm_M3_DIN965"
+		(property "Footprint" "MountingHole:MountingHole_3.2mm_M3_DIN965_Pad"
 			(at 52.07 220.98 0)
 			(effects
@@
 			)
 		)
-		(property "Footprint" "MountingHole:MountingHole_3.2mm_M3_DIN965"
+		(property "Footprint" "MountingHole:MountingHole_3.2mm_M3_DIN965_Pad"
 			(at 52.07 232.41 0)
 			(effects
@@
 			)
 		)
-		(property "Footprint" "Connector_USB:USB_C_Plug_Molex_105444"
+		(property "Footprint" "footprints:CONN_8p94X6p5X3p16_12L_GCC"
 			(at 172.72 261.62 0)
 			(effects
@@
 					(size 1.27 1.27)
 				)
-				(hide yes)
 			)
 		)
@@
 			)
 		)
-		(property "Footprint" ""
+		(property "Footprint" "Button_Switch_SMD:SW_SPST_TS-1088-xR025"
 			(at 161.29 177.8 0)
 			(effects
