File: New Horizons.kicad_pcb (KiCad board)
At the start: 4 copper layers, 18 x 23.3 mm, 280 parts, among them J1 Conn_01x09_Socket, J2 Conn_01x09_Socket, J3 Conn_01x05_Socket, SW1 SW_Push, SW10 SW_Push, SW11 SW_Push, SW12 SW_Push, SW13 SW_Push, SW14 SW_Push, SW15 SW_Push, SW16 SW_Push, SW17 SW_Push, SW18 SW_Push, SW19 SW_Push, SW2 SW_Push, SW20 SW_Push, SW21 SW_Push, SW22 SW_Push, SW23 SW_Push, SW24 SW_Push, SW25 SW_Push, SW26 SW_Push, SW27 SW_Push, SW28 SW_Push, SW29 SW_Push, SW3 SW_Push, SW30 SW_Push, SW31 SW_Push, SW32 SW_Push, SW33 SW_Push, SW34 SW_Push, SW35 SW_Push, SW36 SW_Push, SW37 SW_Push, SW38 SW_Push, SW39 SW_Push, SW4 SW_Push, SW40 SW_Push, SW41 SW_Push, SW42 SW_Push, SW43 SW_Push, SW44 SW_Push, SW45 SW_Push, SW46 SW_Push, SW47 SW_Push, SW48 SW_Push, SW49 SW_Push, SW5 SW_Push, SW50 SW_Push, SW51 SW_Push, SW52 SW_Push, SW53 SW_Push, SW54 SW_Push, SW55 SW_Push, SW56 SW_Push, SW57 SW_Push, SW58 SW_Push, SW59 SW_Push, SW6 SW_Push, SW60 SW_Push, SW61 SW_Push, SW62 SW_Push, SW63 SW_Push, SW64 SW_Push, SW65 SW_Push, SW66 SW_Push, SW67 SW_Push, SW68 SW_Push, SW7 SW_Push, SW8 SW_Push, SW9 SW_Push

Commit message: progress
Parts:
- removed Gemini1: ~, Gemini:gemini
Routing:
- net VCC: track 199.3 -> 794.9 mm, vias 5 -> 9
- net ROW1: track 301.0 -> 359.2 mm
- net ROW0: track 373.5 -> 337.4 mm
- net Net-(LED23-DOUT): track 0.00 -> 14.2 mm
- net GND: track 2.15 -> 13.2 mm, vias 7 -> 0
- net COL15: track 408.5 -> 404.9 mm
- net Net-(LED44-DOUT): track 296.5 -> 300.1 mm
- net COL5: track 175.7 -> 178.0 mm
- net COL6: track 187.2 -> 189.4 mm
- net ROW4: track 403.6 -> 405.9 mm
- net ROW2: track 362.3 -> 364.6 mm
- net COL8: track 233.6 -> 235.9 mm
- net COL13: track 339.2 -> 341.4 mm
- net COL10: track 303.0 -> 305.3 mm
- net COL0: track 90.5 -> 92.7 mm
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- added copper zone on B.Cu, net GND
- added copper zone on F.Cu, net VCC
- removed copper zone on F.Cu, net GND
Other:
- board size 18 x 23.3 mm -> 3.6 x 3.2 mm

Commit message: work
Parts:
- added Gemini1: ~, Gemini:gemini, F.Cu at (-3.78, -49.9)
- added J4: Conn_01x12_Pin, Connector_PinHeader_2.54mm:PinHeader_1x12_P2.54mm_Vertical, F.Cu at (11.5, -48.6)
- J1, J2: value Conn_01x09_Socket -> Conn_01x12_Socket; footprint Connector_PinHeader_2.54mm:PinHeader_1x09_P2.54mm_Vertical -> Connector_PinSocket_2.54mm:PinSocket_1x12_P2.54mm_Vertical
- J3: value Conn_01x05_Socket -> Conn_01x12_Pin; footprint Connector_PinHeader_2.54mm:PinHeader_1x05_P2.54mm_Vertical -> Connector_PinHeader_2.54mm:PinHeader_1x12_P2.54mm_Vertical
- moved J3 74.7 mm to (11.5, -51.3)
- moved J1 28.7 mm to (0.10, -14.1), turned to 90 degrees
- moved J2 13.3 mm to (0.10, -11.1), turned to 90 degrees
Connections:
- J1 pad 1: ROW0 -> ROW4
- J1 pad 2: ROW4 -> ROW3
- J1 pad 3: ROW3 -> ROW2
- J1 pad 4: ROW2 -> ROW1
- J1 pad 5: ROW1 -> ROW0
- J1 pad 6: COL13 -> COL9
- J1 pad 7: COL15 -> COL10
- J1 pad 8: COL14 -> COL11
- J1 pad 9: COL12 -> COL15
- J2 pad 3: COL0 -> unconnected-(J2-Pin_3-Pad3)
- J2 pad 4: COL1 -> COL0
- J2 pad 5: COL2 -> COL1
- J2 pad 6: COL3 -> COL2
- J2 pad 7: COL4 -> COL3
- J2 pad 8: COL5 -> COL4
- J2 pad 9: COL6 -> COL5
- J3 pad 1: COL11 -> ROW4
- J3 pad 2: COL10 -> ROW3
- J3 pad 3: COL9 -> ROW2
- J3 pad 4: COL8 -> ROW1
- J3 pad 5: COL7 -> ROW0
Routing:
- net Net-(LED15-DOUT): track 308.5 -> 0.00 mm
- net ROW3: track 380.9 -> 289.6 mm
- net ROW1: track 359.2 -> 291.3 mm
- net COL1: track 105.7 -> 44.8 mm, vias 2 -> 1
- net COL5: track 178.0 -> 139.3 mm
- net COL6: track 189.4 -> 156.9 mm, vias 5 -> 4
- net COL4: track 152.6 -> 122.5 mm
- net COL3: track 133.5 -> 106.4 mm
- net COL15: track 404.9 -> 377.9 mm
- net COL12: track 351.6 -> 326.1 mm
- net COL14: track 382.4 -> 357.0 mm
- net ROW0: track 337.4 -> 316.0 mm
- net COL11: track 327.3 -> 306.4 mm, vias 6 -> 5
- net COL10: track 305.3 -> 286.2 mm, vias 6 -> 5
- net Net-(LED16-DOUT): track 19.0 -> 0.00 mm
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Other:
- board size 3.6 x 3.2 mm -> 57.9 x 37.8 mm
