File: New Horizons.kicad_pcb (KiCad board)
At the start: 4 copper layers, 57.9 x 37.8 mm, 281 parts, among them J1 Conn_01x12_Socket, J2 Conn_01x12_Socket, J3 Conn_01x12_Pin, J4 Conn_01x12_Pin, SW1 SW_Push, SW10 SW_Push, SW11 SW_Push, SW12 SW_Push, SW13 SW_Push, SW14 SW_Push, SW15 SW_Push, SW16 SW_Push, SW17 SW_Push, SW18 SW_Push, SW19 SW_Push, SW2 SW_Push, SW20 SW_Push, SW21 SW_Push, SW22 SW_Push, SW23 SW_Push, SW24 SW_Push, SW25 SW_Push, SW26 SW_Push, SW27 SW_Push, SW28 SW_Push, SW29 SW_Push, SW3 SW_Push, SW30 SW_Push, SW31 SW_Push, SW32 SW_Push, SW33 SW_Push, SW34 SW_Push, SW35 SW_Push, SW36 SW_Push, SW37 SW_Push, SW38 SW_Push, SW39 SW_Push, SW4 SW_Push, SW40 SW_Push, SW41 SW_Push, SW42 SW_Push, SW43 SW_Push, SW44 SW_Push, SW45 SW_Push, SW46 SW_Push, SW47 SW_Push, SW48 SW_Push, SW49 SW_Push, SW5 SW_Push, SW50 SW_Push, SW51 SW_Push, SW52 SW_Push, SW53 SW_Push, SW54 SW_Push, SW55 SW_Push, SW56 SW_Push, SW57 SW_Push, SW58 SW_Push, SW59 SW_Push, SW6 SW_Push, SW60 SW_Push, SW61 SW_Push, SW62 SW_Push, SW63 SW_Push, SW64 SW_Push, SW65 SW_Push, SW66 SW_Push, SW67 SW_Push, SW68 SW_Push, SW7 SW_Push, SW8 SW_Push, SW9 SW_Push

Commit message: work
Parts:
- J1, J2: moved to B.Cu
- turned J1 to -90 degrees
- turned J2 to -90 degrees
Routing:
- net COL0: track 75.9 -> 140.3 mm, vias 2 -> 4
- net VCC: track 787.4 -> 830.3 mm, vias 5 -> 6
- net ROW0: track 316.0 -> 358.6 mm
- net COL3: track 106.4 -> 141.4 mm, vias 4 -> 5
- net COL4: track 122.5 -> 157.1 mm, vias 4 -> 5
- net COL5: track 139.3 -> 173.4 mm, vias 4 -> 5
- net COL6: track 156.9 -> 189.5 mm
- net ROW3: track 289.6 -> 322.0 mm, vias 13 -> 14
- net ROW4: track 396.8 -> 428.7 mm
- net ROW2: track 365.1 -> 395.9 mm, vias 14 -> 15
- net ROW1: track 291.3 -> 321.5 mm, vias 15 -> 16
- net GND: track 25.4 -> 38.7 mm, vias 0 -> 1
- net COL7: track 224.2 -> 227.0 mm, vias 5 -> 6
- net COL10: track 286.2 -> 288.9 mm
- net COL12: track 326.1 -> 328.3 mm
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Other:
- board size 57.9 x 37.8 mm -> 312.2 x 154.4 mm
