File: New Horizons.kicad_pcb (KiCad board)
At the start: 4 copper layers, 312.2 x 154.4 mm, 281 parts, among them J1 Conn_01x12_Socket, J2 Conn_01x12_Socket, J3 Conn_01x12_Pin, J4 Conn_01x12_Pin, SW1 SW_Push, SW10 SW_Push, SW11 SW_Push, SW12 SW_Push, SW13 SW_Push, SW14 SW_Push, SW15 SW_Push, SW16 SW_Push, SW17 SW_Push, SW18 SW_Push, SW19 SW_Push, SW2 SW_Push, SW20 SW_Push, SW21 SW_Push, SW22 SW_Push, SW23 SW_Push, SW24 SW_Push, SW25 SW_Push, SW26 SW_Push, SW27 SW_Push, SW28 SW_Push, SW29 SW_Push, SW3 SW_Push, SW30 SW_Push, SW31 SW_Push, SW32 SW_Push, SW33 SW_Push, SW34 SW_Push, SW35 SW_Push, SW36 SW_Push, SW37 SW_Push, SW38 SW_Push, SW39 SW_Push, SW4 SW_Push, SW40 SW_Push, SW41 SW_Push, SW42 SW_Push, SW43 SW_Push, SW44 SW_Push, SW45 SW_Push, SW46 SW_Push, SW47 SW_Push, SW48 SW_Push, SW49 SW_Push, SW5 SW_Push, SW50 SW_Push, SW51 SW_Push, SW52 SW_Push, SW53 SW_Push, SW54 SW_Push, SW55 SW_Push, SW56 SW_Push, SW57 SW_Push, SW58 SW_Push, SW59 SW_Push, SW6 SW_Push, SW60 SW_Push, SW61 SW_Push, SW62 SW_Push, SW63 SW_Push, SW64 SW_Push, SW65 SW_Push, SW66 SW_Push, SW67 SW_Push, SW68 SW_Push, SW7 SW_Push, SW8 SW_Push, SW9 SW_Push

Commit message: work
Parts:
- moved J4 15.1 mm to (-0.41, -57.8)
- moved J3 15.0 mm to (-0.41, -60.4)
- moved Gemini1 5.62 mm to (-0.09, -45.7)
- moved J1 0.44 mm to (0.10, -13.7)
Routing:
- net COL13: track 323.4 -> 279.3 mm
- net VCC: track 830.3 -> 787.4 mm, vias 6 -> 5
- net ROW0: track 358.6 -> 316.0 mm
- net GND: track 38.7 -> 0.00 mm, vias 1 -> 0
- net COL12: track 328.3 -> 290.7 mm, vias 6 -> 5
- net COL14: track 356.3 -> 319.2 mm
- net COL2: track 147.4 -> 110.8 mm
- net COL15: track 377.0 -> 341.0 mm
- net COL1: track 45.2 -> 9.27 mm
- net COL3: track 141.4 -> 106.4 mm, vias 5 -> 4
- net COL7: track 227.0 -> 192.1 mm, vias 6 -> 5
- net COL0: track 140.3 -> 105.6 mm
- net COL4: track 157.1 -> 122.5 mm, vias 5 -> 4
- net COL8: track 222.2 -> 187.7 mm
- net COL5: track 173.4 -> 139.3 mm, vias 5 -> 4
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