File: New Horizons.kicad_sch (KiCad schematic)
At the start: 0 parts

Commit message: progress
Other:
- added sheet Controller Board (Controller Board.kicad_sch)
Changed lines of the file:
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@@
+	)
+	(sheet
+		(at 22.225 61.595)
+		(size 22.86 15.24)
+		(exclude_from_sim no)
+		(in_bom yes)
+		(on_board yes)
+		(dnp no)
+		(fields_autoplaced yes)
+		(stroke
+			(width 0.1524)
+			(type solid)
+		)
+		(fill
+			(color 0 0 0 0)
+		)
+		(property "Sheetname" "Controller Board"
+			(at 22.225 60.8834 0)
+			(show_name no)
+			(do_not_autoplace no)
+			(effects
+				(font
+					(size 1.27 1.27)
+				)
+				(justify left bottom)
+			)
+		)
+		(property "Sheetfile" "Controller Board.kicad_sch"
+			(at 22.225 77.4196 0)
+			(show_name no)
+			(do_not_autoplace no)
+			(effects
+				(font
+					(size 1.27 1.27)
+				)
+				(justify left top)
+			)
+		)
+		(instances
+			(project "New Horizons"
+				(path "/e965cafa-4916-4eb8-baa0-65aec817bdb5"
+					(page "4")
+				)
+			)
+		)
 	)
 	(sheet
