File: Main Board.kicad_pcb (KiCad board)
At the start: 4 copper layers, 308 x 103.6 mm, 277 parts, among them J1 Conn_01x12_Socket, J2 Conn_01x12_Socket, SW1 SW_Push, SW10 SW_Push, SW11 SW_Push, SW12 SW_Push, SW13 SW_Push, SW14 SW_Push, SW15 SW_Push, SW16 SW_Push, SW17 SW_Push, SW18 SW_Push, SW19 SW_Push, SW2 SW_Push, SW20 SW_Push, SW21 SW_Push, SW22 SW_Push, SW23 SW_Push, SW24 SW_Push, SW25 SW_Push, SW26 SW_Push, SW27 SW_Push, SW28 SW_Push, SW29 SW_Push, SW3 SW_Push, SW30 SW_Push, SW31 SW_Push, SW32 SW_Push, SW33 SW_Push, SW34 SW_Push, SW35 SW_Push, SW36 SW_Push, SW37 SW_Push, SW38 SW_Push, SW39 SW_Push, SW4 SW_Push, SW40 SW_Push, SW41 SW_Push, SW42 SW_Push, SW43 SW_Push, SW44 SW_Push, SW45 SW_Push, SW46 SW_Push, SW47 SW_Push, SW48 SW_Push, SW49 SW_Push, SW5 SW_Push, SW50 SW_Push, SW51 SW_Push, SW52 SW_Push, SW53 SW_Push, SW54 SW_Push, SW55 SW_Push, SW56 SW_Push, SW57 SW_Push, SW58 SW_Push, SW59 SW_Push, SW6 SW_Push, SW60 SW_Push, SW61 SW_Push, SW62 SW_Push, SW63 SW_Push, SW64 SW_Push, SW65 SW_Push, SW66 SW_Push, SW67 SW_Push, SW68 SW_Push, SW7 SW_Push, SW8 SW_Push, SW9 SW_Push

Commit message: checkpoint
Parts:
- moved D29 3.30 mm to (270.7, 14.6)
- moved D37 3.30 mm to (137.4, 33.6)
- moved D38 3.30 mm to (156.4, 33.6)
- moved D39 3.30 mm to (175.5, 33.6)
- moved D40 3.30 mm to (194.5, 33.6)
- moved D41 3.30 mm to (213.6, 33.6)
- moved D42 3.30 mm to (232.6, 33.6)
- moved D51 3.30 mm to (146.9, 52.6)
- moved D52 3.30 mm to (166.0, 52.6)
- moved D53 3.30 mm to (185.0, 52.6)
- moved D55 3.30 mm to (223.1, 52.6)
- moved D43 3.30 mm to (263.6, 33.6)
- moved D62 3.30 mm to (130.2, 71.7)
- moved D45 3.30 mm to (20.7, 52.6)
- moved D10 3.30 mm to (180.2, -4.50)
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
Commit message: checkpoint
Routing:
- net ROW1: track 347.2 -> 46.2 mm, vias 14 -> 0
- net ROW2: track 364.7 -> 65.6 mm, vias 14 -> 0
- net Net-(D13-A): track 0.00 -> 48.5 mm
- net Net-(D9-A): track 0.00 -> 28.9 mm
- net Net-(D8-A): track 0.00 -> 27.3 mm
- net Net-(D2-A): track 0.00 -> 27.1 mm
- net Net-(D61-A): track 0.00 -> 3.56 mm
- net Net-(D5-A): track 0.00 -> 3.55 mm
- net Net-(D3-A): track 0.00 -> 3.55 mm
- net Net-(D1-A): track 0.00 -> 3.55 mm
- net Net-(D65-A): track 0.00 -> 3.55 mm
- net Net-(D63-A): track 0.00 -> 3.55 mm
- net Net-(D7-A): track 0.00 -> 3.55 mm
- net Net-(D67-A): track 0.00 -> 3.55 mm
- net Net-(D15-A): track 0.00 -> 3.55 mm
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