File: Main Board.kicad_pcb (KiCad board)
At the start: 4 copper layers, 308 x 103.6 mm, 277 parts, among them J1 Conn_01x12_Socket, J2 Conn_01x12_Socket, SW1 SW_Push, SW10 SW_Push, SW11 SW_Push, SW12 SW_Push, SW13 SW_Push, SW14 SW_Push, SW15 SW_Push, SW16 SW_Push, SW17 SW_Push, SW18 SW_Push, SW19 SW_Push, SW2 SW_Push, SW20 SW_Push, SW21 SW_Push, SW22 SW_Push, SW23 SW_Push, SW24 SW_Push, SW25 SW_Push, SW26 SW_Push, SW27 SW_Push, SW28 SW_Push, SW29 SW_Push, SW3 SW_Push, SW30 SW_Push, SW31 SW_Push, SW32 SW_Push, SW33 SW_Push, SW34 SW_Push, SW35 SW_Push, SW36 SW_Push, SW37 SW_Push, SW38 SW_Push, SW39 SW_Push, SW4 SW_Push, SW40 SW_Push, SW41 SW_Push, SW42 SW_Push, SW43 SW_Push, SW44 SW_Push, SW45 SW_Push, SW46 SW_Push, SW47 SW_Push, SW48 SW_Push, SW49 SW_Push, SW5 SW_Push, SW50 SW_Push, SW51 SW_Push, SW52 SW_Push, SW53 SW_Push, SW54 SW_Push, SW55 SW_Push, SW56 SW_Push, SW57 SW_Push, SW58 SW_Push, SW59 SW_Push, SW6 SW_Push, SW60 SW_Push, SW61 SW_Push, SW62 SW_Push, SW63 SW_Push, SW64 SW_Push, SW65 SW_Push, SW66 SW_Push, SW67 SW_Push, SW68 SW_Push, SW7 SW_Push, SW8 SW_Push, SW9 SW_Push

Commit message: checkpoint
Parts:
- added D18: D, Diode_SMD:D_SOD-123, B.Cu at (55.6, 18.6)
- SW1, SW10, SW11, SW12, SW13, SW14, SW15, SW16, SW17, SW18, SW19, SW2, SW20, SW21, SW22, SW23, SW24, SW25, SW26, SW27, SW28, SW29, SW3, SW30, SW31, SW32, SW33, SW34, SW35, SW36, SW37, SW38, SW39, SW4, SW40, SW41, SW42, SW43, SW44, SW45, SW46, SW47, SW48, SW49, SW5, SW50, SW51, SW52, SW53, SW54, SW55, SW56, SW57, SW58, SW59, SW6, SW60, SW61, SW62, SW63, SW64, SW65, SW66, SW67, SW68, SW7, SW8, SW9: footprint PCM_Switch_Keyboard_Hotswap_Kailh:SW_Hotswap_Kailh_MX -> mx_hotswap:MX-Hotswap-1U; moved to B.Cu
- moved D44 4.20 mm to (293.6, 37.7)
- moved D57 4.20 mm to (274.6, 56.7)
- moved D58 4.20 mm to (293.6, 56.7)
- moved D14 4.20 mm to (265.0, -0.41)
- moved D15 4.20 mm to (293.6, -0.41)
- moved D30 4.20 mm to (293.6, 18.6)
- moved D31 4.20 mm to (10.2, 37.7)
- moved D32 4.20 mm to (41.2, 37.7)
- moved D33 4.20 mm to (60.2, 37.7)
- moved D34 4.20 mm to (79.3, 37.7)
- moved D35 4.20 mm to (98.3, 37.7)
- moved D36 4.20 mm to (117.4, 37.7)
- moved D37 4.20 mm to (136.4, 37.7)
- moved D38 4.20 mm to (155.5, 37.7)
- moved D39 4.20 mm to (174.5, 37.7)
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Routing:
- net Net-(LED30-DOUT): track 306.7 -> 0.00 mm
- net Net-(LED58-DOUT): track 305.9 -> 0.00 mm
- net Net-(LED15-DOUT): track 304.7 -> 0.00 mm
- net ROW2: track 65.6 -> 350.9 mm, vias 0 -> 14
- net ROW1: track 46.2 -> 330.9 mm, vias 0 -> 15
- net COL13: track 291.6 -> 72.2 mm, vias 4 -> 3
- net COL12: track 294.4 -> 92.4 mm
- net Net-(D13-A): track 48.5 -> 3.86 mm
- net Net-(D9-A): track 28.9 -> 3.86 mm
- net Net-(D8-A): track 27.3 -> 3.86 mm
- net Net-(D2-A): track 27.1 -> 3.86 mm
- net ROW4: track 389.8 -> 396.9 mm
- net GND: track 42.5 -> 36.9 mm
- net Net-(D18-A): track 0.00 -> 3.87 mm
- net Net-(D68-A): track 3.53 -> 0.00 mm
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
Commit message: checkpoint
Parts:
- removed ST14, ST43, ST45: SW_stab, Mounting_Keyboard_Stabilizer:Stabilizer_Cherry_MX_2.00u
- removed ST62: SW_stab, Mounting_Keyboard_Stabilizer:Stabilizer_Cherry_MX_6.25u
- added Gemini1: ~, Gemini:gemini, F.Cu at (20.3, -56.3)
- added J3: Conn_01x12_Header, Connector_PinHeader_2.54mm:PinHeader_1x12_P2.54mm_Vertical, B.Cu at (18.4, -75.2)
- added J4: Conn_01x12_Header, Connector_PinHeader_2.54mm:PinHeader_1x12_P2.54mm_Vertical, B.Cu at (18.4, -71.6)
- J1, J2: value Conn_01x12_Socket -> Conn_01x12_Pin
- moved J2 0.06 mm to (0.10, -11.2)
Routing:
- net Net-(LED58-DOUT): track 0.00 -> 302.8 mm, vias 0 -> 2
- net Net-(LED30-DOUT): track 0.00 -> 302.8 mm, vias 0 -> 2
- net Net-(LED15-DOUT): track 0.00 -> 300.4 mm, vias 0 -> 2
- net COL13: track 72.2 -> 291.0 mm
- net COL12: track 92.4 -> 290.9 mm
- net _COL0: track 0.00 -> 49.7 mm, vias 0 -> 1
- net _COL1: track 0.00 -> 45.7 mm, vias 0 -> 1
- net _COL2: track 0.00 -> 41.6 mm, vias 0 -> 1
- net _COL3: track 0.00 -> 38.6 mm, vias 0 -> 1
- net _COL4: track 0.00 -> 37.2 mm, vias 0 -> 1
- net _COL5: track 0.00 -> 34.4 mm, vias 0 -> 1
- net _COL12: track 0.00 -> 31.8 mm
- net _COL13: track 0.00 -> 31.2 mm
- net _COL6: track 0.00 -> 30.3 mm, vias 0 -> 1
- net _COL8: track 0.00 -> 28.8 mm
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Other:
- board size 308 x 103.6 mm -> 309 x 171 mm
