File: Main Board.kicad_pcb (KiCad board)
At the start: 4 copper layers, 309 x 171 mm, 277 parts, among them J1 Conn_01x12_Pin, J2 Conn_01x12_Pin, J3 Conn_01x12_Header, J4 Conn_01x12_Header, SW1 SW_Push, SW10 SW_Push, SW11 SW_Push, SW12 SW_Push, SW13 SW_Push, SW14 SW_Push, SW15 SW_Push, SW16 SW_Push, SW17 SW_Push, SW18 SW_Push, SW19 SW_Push, SW2 SW_Push, SW20 SW_Push, SW21 SW_Push, SW22 SW_Push, SW23 SW_Push, SW24 SW_Push, SW25 SW_Push, SW26 SW_Push, SW27 SW_Push, SW28 SW_Push, SW29 SW_Push, SW3 SW_Push, SW30 SW_Push, SW31 SW_Push, SW32 SW_Push, SW33 SW_Push, SW34 SW_Push, SW35 SW_Push, SW36 SW_Push, SW37 SW_Push, SW38 SW_Push, SW39 SW_Push, SW4 SW_Push, SW40 SW_Push, SW41 SW_Push, SW42 SW_Push, SW43 SW_Push, SW44 SW_Push, SW45 SW_Push, SW46 SW_Push, SW47 SW_Push, SW48 SW_Push, SW49 SW_Push, SW5 SW_Push, SW50 SW_Push, SW51 SW_Push, SW52 SW_Push, SW53 SW_Push, SW54 SW_Push, SW55 SW_Push, SW56 SW_Push, SW57 SW_Push, SW58 SW_Push, SW59 SW_Push, SW6 SW_Push, SW60 SW_Push, SW61 SW_Push, SW62 SW_Push, SW63 SW_Push, SW64 SW_Push, SW65 SW_Push, SW66 SW_Push, SW67 SW_Push, SW68 SW_Push, SW7 SW_Push, SW8 SW_Push, SW9 SW_Push

Commit message: checkpoint w gemini routed
Parts:
- added U1: ProMicro, keebio:Elite-C, F.Cu at (18.0, 9.08)
Connections:
- J1 pad 12: COL12 -> COL15
- J1 pad 9: COL15 -> COL12
- J2 pad 3: unconnected-(J2-Pin_3-Pad3) -> COL0
- J2 pad 4: COL0 -> ROW3
- J4 pad 3: unconnected-(J4-Pin_3-Pad3) -> _LEDIN
Routing:
- net VCC: track 150.9 -> 223.1 mm, vias 0 -> 2
- net GND: track 37.4 -> 101.8 mm, vias 136 -> 138
- net LEDIN: track 0.00 -> 28.6 mm
- net COL12: track 290.9 -> 298.6 mm, vias 5 -> 6
- net COL15: track 339.5 -> 332.2 mm, vias 6 -> 5
- net ROW3: track 365.5 -> 359.0 mm
- net _COL11: track 19.6 -> 25.1 mm
- net _COL10: track 19.8 -> 24.6 mm
- net COL13: track 291.0 -> 294.2 mm
- net _COL9: track 21.9 -> 24.5 mm
- net COL0: track 105.5 -> 103.0 mm
- net _COL15: track 23.5 -> 25.6 mm
- net _COL13: track 31.2 -> 33.1 mm
- net _ROW1: track 12.8 -> 13.9 mm
- net _COL14: track 20.6 -> 21.3 mm
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
Commit message: use pro micro over gemini
Parts:
- removed Gemini1: ~, Gemini:gemini
- J3, J4: moved to F.Cu
- U1: value ProMicro -> ~; footprint keebio:Elite-C -> kicad_pro_micro_rp2040:pro_micro_rp2040
- moved U1 49.3 mm to (34.4, -37.5), turned to 90 degrees
- moved J3 11.0 mm to (13.5, -65.4), turned to 90 degrees
- moved J4 11.0 mm to (13.5, -61.8), turned to 90 degrees
Connections:
- J1 pad 2: ROW3 -> LEDIN
- J2 pad 3: COL0 -> ROW3
- J4 pad 1: VCC -> _VCC
- J4 pad 2: GND -> _GND
- U1 pad 11: unconnected-(U1-8/B4-Pad11) -> _LEDIN
- U1 pad 12: unconnected-(U1-9/B5-Pad12) -> _COL7
- U1 pad 13: unconnected-(U1-B6/10-Pad13) -> _COL12
- U1 pad 14: unconnected-(U1-B2/16-Pad14) -> _COL13
- U1 pad 15: unconnected-(U1-B3/14-Pad15) -> _COL14
- U1 pad 16: unconnected-(U1-B1/15-Pad16) -> _COL15
- U1 pad 2: unconnected-(U1-RX1/D2-Pad2) -> _COL0
- U1 pad 20: unconnected-(U1-F4/A3-Pad20) -> _COL9
- U1 pad 21: VCC -> _COL11
- U1 pad 22: unconnected-(U1-RST-Pad22) -> _ROW0
- U1 pad 23: GND -> _COL10
- U1 pad 25: (no net) -> unconnected-(U1-GP25-Pad25)
- U1 pad 26: (no net) -> _ROW1
- U1 pad 27: (no net) -> _ROW2
- U1 pad 28: (no net) -> _ROW3
- U1 pad 29: (no net) -> _ROW4
- U1 pad 3: GND -> _COL1
- U1 pad 4: GND -> _COL2
- U1 pad 5: unconnected-(U1-2/D1/SDA-Pad5) -> _COL3
- U1 pad 6: unconnected-(U1-3/D0/SCL-Pad6) -> _COL4
- U1 pad 7: unconnected-(U1-4/D4-Pad7) -> _COL5
- U1 pad 8: unconnected-(U1-5/C6-Pad8) -> _COL6
- U1 pad 9: unconnected-(U1-6/D7-Pad9) -> _COL8
Routing:
- net VCC: track 223.1 -> 150.9 mm, vias 2 -> 0
- net GND: track 101.8 -> 37.4 mm, vias 138 -> 136
- net _GND: track 0.00 -> 45.3 mm
- net _COL0: track 49.7 -> 27.2 mm, vias 1 -> 0
- net _LEDIN: track 0.00 -> 20.2 mm
- net _COL1: track 45.7 -> 25.5 mm, vias 1 -> 0
- net _COL2: track 41.7 -> 25.5 mm, vias 1 -> 0
- net _COL3: track 38.6 -> 25.6 mm, vias 1 -> 0
- net _COL11: track 25.1 -> 12.2 mm, vias 1 -> 0
- net _COL10: track 24.6 -> 12.2 mm, vias 1 -> 0
- net _COL9: track 24.5 -> 12.2 mm, vias 1 -> 0
- net _ROW0: track 23.9 -> 12.2 mm
- net _VCC: track 0.00 -> 11.6 mm
- net _COL4: track 36.8 -> 25.5 mm, vias 1 -> 0
- net _COL13: track 33.1 -> 22.4 mm
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Other:
- board size 309 x 171 mm -> 309 x 161.2 mm
