File: Main Board.kicad_sch (KiCad schematic)
At the start: 0 parts

Commit message: checkpoint
Other:
- sheet Key Matrix: file New Horizons-key-matrix.kicad_sch -> key-matrix.kicad_sch
- sheet Led Chain: file New Horizons-led-chain.kicad_sch -> led-chain.kicad_sch
Changed lines of the file:
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@@
 			)
 		)
-		(property "Sheetfile" "New Horizons-led-chain.kicad_sch"
+		(property "Sheetfile" "led-chain.kicad_sch"
 			(at 21.59 52.9696 0)
 			(show_name no)
@@
 		)
 		(instances
-			(project "New Horizons"
+			(project "Main Board"
 				(path "/e965cafa-4916-4eb8-baa0-65aec817bdb5"
 					(page "3")
@@
 		)
 		(instances
-			(project "New Horizons"
+			(project "Main Board"
 				(path "/e965cafa-4916-4eb8-baa0-65aec817bdb5"
 					(page "4")
@@
 			)
 		)
-		(property "Sheetfile" "New Horizons-key-matrix.kicad_sch"
+		(property "Sheetfile" "key-matrix.kicad_sch"
 			(at 21.59 32.9696 0)
 			(show_name no)
@@
 		)
 		(instances
-			(project "New Horizons"
+			(project "Main Board"
 				(path "/e965cafa-4916-4eb8-baa0-65aec817bdb5"
 					(page "2")
